Commit message: Gazebo configuration done along with colors

File: description/robot_core.xacro (robot description, xacro)
@@ -41,4 +41,7 @@
     </xacro:inertial_box>
 </link>
+<gazebo reference="chassis">
+    <material>Gazebo/White</material>
+</gazebo>
 <!-- Left Wheel Link -->
 <joint name="left_wheel_joint" type="continuous">
@@ -66,4 +69,7 @@
     </xacro:inertial_cylinder>
 </link>
+<gazebo reference="left_wheel">
+    <material>Gazebo/Blue</material>
+</gazebo>
 <!-- Right Wheel Link -->
 <joint name="right_wheel_joint" type="continuous">
@@ -91,4 +97,7 @@
     </xacro:inertial_cylinder>
 </link>
+<gazebo reference="right_wheel">
+    <material>Gazebo/Blue</material>
+</gazebo>
 <!-- Castor Wheel Link -->
 <joint name="castor_wheel_joint" type="fixed">
@@ -115,3 +124,6 @@
     </xacro:inertial_sphere>
 </link>
+<gazebo reference="castor_wheel">
+    <material>Gazebo/Black</material>
+</gazebo>
 </robot>
